Commit message: Add YOLOv8 stairs detection, Gazebo staircase and CI
- Detect stairs with yolov8n-oiv7 (Open Images, has a Stairs class);
  the model is cached in a fixed directory so it also loads under systemd
- Pin numpy<2 so ROS 2 Jazzy cv_bridge works alongside ultralytics
- Gazebo: staircase, indoor lighting, hazard guard in the command path
  and an optional detector
- CI workflow for the ROS 2 packages and the firmware

File: ros2_ws/src/amr_description/urdf/amr.urdf.xacro (robot description, xacro)
@@ -1,5 +1,6 @@
 <?xml version="1.0"?>
-<!-- AMR: 80 x 45 cm aluminium tube frame, two wiper-motor drive wheels on the centre axle,
-     four swivel casters at the corners, RPLidar in the exact centre, forward camera, top deck.
+<!-- AMR: 80 x 45 cm aluminium tube frame, two wiper-motor drive wheels 20 cm from the rear,
+     two swivel casters at the front corners, RPLidar in the exact centre of the frame,
+     forward camera, top deck. base_link is the midpoint of the drive axle (the turning centre).
      Dimensions match amr_sim/worlds/amr_world.sdf and amr_base/config/base.yaml. -->
 <robot name="amr" xmlns:xacro="http://www.ros.org/wiki/xacro">
@@ -9,10 +10,12 @@
   <xacro:property name="wheel_radius" value="0.075"/>
   <xacro:property name="wheel_separation" value="0.30"/>
+  <xacro:property name="axle_to_front" value="0.60"/>     <!-- drive axle is 60 cm behind the front edge -->
   <!-- Estimated from photos: re-measure and adjust -->
   <xacro:property name="chassis_z" value="0.05"/>        <!-- frame tube height -->
   <xacro:property name="wheel_width" value="0.04"/>
-  <xacro:property name="caster_x" value="0.35"/>         <!-- caster centres from robot centre -->
+  <xacro:property name="caster_inset" value="0.05"/>     <!-- caster centre from the front edge -->
   <xacro:property name="caster_y" value="0.18"/>
   <xacro:property name="deck_height" value="0.17"/>      <!-- top deck above base_link -->
+  <xacro:property name="frame_x" value="${axle_to_front - chassis_x/2}"/>  <!-- frame centre, 0.2 m ahead of the axle -->
   <xacro:property name="lidar_height" value="0.10"/>     <!-- scan plane above base_link: clears the tyre tops -->
   <material name="frame"><color rgba="0.12 0.12 0.12 1"/></material>
@@ -28,14 +31,22 @@
     </inertial>
   </xacro:macro>
-  <!-- base_link: centre of the frame, on the drive axle, one wheel radius above the floor -->
+  <!-- base_link: midpoint of the drive axle, one wheel radius above the floor -->
   <link name="base_link">
     <visual>
+      <origin xyz="${frame_x} 0 0"/>
       <geometry><box size="${chassis_x} ${chassis_y} ${chassis_z}"/></geometry>
       <material name="frame"/>
     </visual>
     <collision>
+      <origin xyz="${frame_x} 0 0"/>
       <geometry><box size="${chassis_x} ${chassis_y} ${chassis_z}"/></geometry>
     </collision>
-    <xacro:box_inertia m="8.0" x="${chassis_x}" y="${chassis_y}" z="${chassis_z}"/>
+    <inertial>
+      <origin xyz="${frame_x} 0 0"/>
+      <mass value="8.0"/>
+      <inertia ixx="${8.0*(chassis_y*chassis_y+chassis_z*chassis_z)/12}" ixy="0" ixz="0"
+               iyy="${8.0*(chassis_x*chassis_x+chassis_z*chassis_z)/12}" iyz="0"
+               izz="${8.0*(chassis_x*chassis_x+chassis_y*chassis_y)/12}"/>
+    </inertial>
   </link>
   <link name="base_footprint"/>
@@ -54,5 +65,5 @@
     <parent link="base_link"/>
     <child link="deck"/>
-    <origin xyz="0 0 ${deck_height}"/>
+    <origin xyz="${frame_x} 0 ${deck_height}"/>
   </joint>
   <xacro:macro name="wheel" params="side y">
@@ -95,9 +106,7 @@
     </joint>
   </xacro:macro>
-  <xacro:caster name="front_left" x="${caster_x}" y="${caster_y}"/>
-  <xacro:caster name="front_right" x="${caster_x}" y="${-caster_y}"/>
-  <xacro:caster name="rear_left" x="${-caster_x}" y="${caster_y}"/>
-  <xacro:caster name="rear_right" x="${-caster_x}" y="${-caster_y}"/>
-  <!-- RPLidar A1 in the exact centre of the robot -->
+  <xacro:caster name="front_left" x="${axle_to_front - caster_inset}" y="${caster_y}"/>
+  <xacro:caster name="front_right" x="${axle_to_front - caster_inset}" y="${-caster_y}"/>
+  <!-- RPLidar A1 in the exact centre of the frame -->
   <link name="lidar_link">
     <visual>
@@ -109,7 +118,7 @@
     <parent link="base_link"/>
     <child link="lidar_link"/>
-    <origin xyz="0 0 ${lidar_height}"/>
+    <origin xyz="${frame_x} 0 ${lidar_height}"/>
   </joint>
-  <!-- Forward camera on the front cross-member, tilted down ~20° to see floor edges and stairs -->
+  <!-- Forward camera on the front edge of the top deck, tilted down ~7° to see stairs and floor edges -->
   <link name="camera_link">
     <visual>
@@ -121,5 +130,5 @@
     <parent link="base_link"/>
     <child link="camera_link"/>
-    <origin xyz="${chassis_x/2} 0 0.05" rpy="0 0.35 0"/>
+    <origin xyz="${axle_to_front} 0 ${deck_height}" rpy="0 0.12 0"/>
   </joint>
   <!-- Optical frame (z forward, x right) for image consumers -->

Commit message: Add simulation demos and a shared robot model
- Gazebo uses the same URDF as the robot, with wheel joint states
- Nav2 footprint offset from the drive axle for the 80 x 45 cm body
- Clean Nav2 RViz view for the sim and for the laptop on the real robot
- README demos: SLAM + Nav2 patrol, YOLOv8 stairs stop
- Docker/Pi: CPU-only PyTorch, setuptools pinned to keep pkg_resources

File: ros2_ws/src/amr_description/urdf/amr.urdf.xacro (robot description, xacro)
@@ -1,21 +1,21 @@
 <?xml version="1.0"?>
-<!-- AMR: 80 x 45 cm aluminium tube frame, two wiper-motor drive wheels 20 cm from the rear,
-     two swivel casters at the front corners, RPLidar in the exact centre of the frame,
+<!-- AMR: 80 x 45 cm aluminium tube frame, two wiper-motor drive wheels 20 cm behind the front,
+     two swivel casters at the rear corners, RPLidar in the exact centre of the frame,
      forward camera, top deck. base_link is the midpoint of the drive axle (the turning centre).
      Dimensions match amr_sim/worlds/amr_world.sdf and amr_base/config/base.yaml. -->
 <robot name="amr" xmlns:xacro="http://www.ros.org/wiki/xacro">
-  <!-- Measured -->
+  <!-- Main dimensions -->
   <xacro:property name="chassis_x" value="0.80"/>
   <xacro:property name="chassis_y" value="0.45"/>
   <xacro:property name="wheel_radius" value="0.075"/>
   <xacro:property name="wheel_separation" value="0.30"/>
-  <xacro:property name="axle_to_front" value="0.60"/>     <!-- drive axle is 60 cm behind the front edge -->
-  <!-- Estimated from photos: re-measure and adjust -->
+  <xacro:property name="axle_to_front" value="0.20"/>     <!-- drive axle is 60 cm from the rear edge -->
+  <!-- Frame, caster and sensor mounting details -->
   <xacro:property name="chassis_z" value="0.05"/>        <!-- frame tube height -->
   <xacro:property name="wheel_width" value="0.04"/>
-  <xacro:property name="caster_inset" value="0.05"/>     <!-- caster centre from the front edge -->
+  <xacro:property name="caster_inset" value="0.05"/>     <!-- caster centre from the rear edge -->
   <xacro:property name="caster_y" value="0.18"/>
   <xacro:property name="deck_height" value="0.17"/>      <!-- top deck above base_link -->
-  <xacro:property name="frame_x" value="${axle_to_front - chassis_x/2}"/>  <!-- frame centre, 0.2 m ahead of the axle -->
+  <xacro:property name="frame_x" value="${axle_to_front - chassis_x/2}"/>  <!-- frame centre, 0.2 m behind the axle -->
   <xacro:property name="lidar_height" value="0.10"/>     <!-- scan plane above base_link: clears the tyre tops -->
   <material name="frame"><color rgba="0.12 0.12 0.12 1"/></material>
@@ -106,6 +106,6 @@
     </joint>
   </xacro:macro>
-  <xacro:caster name="front_left" x="${axle_to_front - caster_inset}" y="${caster_y}"/>
-  <xacro:caster name="front_right" x="${axle_to_front - caster_inset}" y="${-caster_y}"/>
+  <xacro:caster name="rear_left" x="${axle_to_front - chassis_x + caster_inset}" y="${caster_y}"/>
+  <xacro:caster name="rear_right" x="${axle_to_front - chassis_x + caster_inset}" y="${-caster_y}"/>
   <!-- RPLidar A1 in the exact centre of the frame -->
   <link name="lidar_link">
